Commit message: change mesh path to relative path for parsing by urdfpy library

File: setup_3_support/urdf/work/halfopen_box.urdf (robot description, URDF)
Before this commit: robot halfopen_box, 2 links, 1 joints
Links:
- link wobj: geometry collision mesh filename=halfopen_box.stl scale=.001 .001 .001; visual mesh filename=halfopen_box.stl scale=.001 .001 .001
Joints:
- joint work_to_wobj: origin xyz=1 1 0 rpy=0 0 ${radians(90)} -> xyz=1 1 0 rpy=0 0 1.5707963267948966
