Commit message: add moveit config

File: setup_3_support/urdf/setup_3.xacro (robot description, xacro)
@@ -90,8 +90,9 @@
 </joint> -->
 <link name="work"/>
-<joint name="table_to_wobj" type="fixed">
+<joint name="table_to_work" type="fixed">
   <parent link="table"/>
   <child link="work"/>
   <origin xyz="-0.5 0.3 0" rpy="0 0 0" />
 </joint>
+<!-- <xacro:include filename="$(find setup_3_support)/urdf/work/halfopen_box.urdf" /> -->
 </robot>

Commit message: fix robot model setup 3

File: setup_3_support/urdf/setup_3.xacro (robot description, xacro)
@@ -39,5 +39,5 @@
     </collision>
 </link>
-<!-- <link name="torch_tip"/> -->
+<link name="torch_tip"/>
 <link name="tool_tip"/>
 <joint name="tool0_to_torch" type="fixed">
@@ -46,15 +46,15 @@
     <child link="torch"/>
 </joint>
-<joint name="torch_to_tool_tip" type="fixed">
+<joint name="torch_to_torch_tip" type="fixed">
     <parent link="torch"/>
-    <child link="tool_tip"/>
+    <child link="torch_tip"/>
     <origin xyz="0.315 0 0.035" rpy="0 2.3560569232 0" />
 </joint>
 <!-- weld tip offset from workpiece -->
-<!-- <joint name="torch_tip_to_tool_tip" type="fixed">
+<joint name="torch_tip_to_tool_tip" type="fixed">
     <parent link="torch_tip"/>
     <child link="tool_tip"/>
-    <origin xyz="0 0 0" rpy="0 0 0" />
-</joint> -->
+    <origin xyz="0 0 0.05" rpy="0 0 0" />
+</joint>
 <!-- Rotation table
 Connects to world with link        "table_base"
