Commit message: add extra box to kingpin case

File: setup_1_support/scripts/templates/workobject.template.urdf (robot description, URDF)
Before this commit: robot $name, 0 links, 0 joints
Links:
- added link world

File: setup_1_support/urdf/work/kingpin.urdf (robot description, URDF)
Before this commit: robot kingpin, 6 links, 5 joints
Links:
- added link u_profile_2; collision box size=0.2 0.5 0.1; visual box size=0.2 0.5 0.1
- link obstacle: geometry collision box size=0.2 0.0833333333333 0.01; visual box size=0.2 0.0833333333333 0.01
- link side_1: geometry collision box size=0.3 0.1 0.055; visual box size=0.3 0.1 0.055
- link side_2: geometry collision box size=0.3 0.1 0.055; visual box size=0.3 0.1 0.055
- link table: geometry collision box size=0.7 0.7 0.01; visual box size=0.7 0.7 0.01
- link u_profile: geometry collision box size=0.2 0.5 0.1; visual box size=0.2 0.5 0.1
Joints:
- added joint world_to_u_profile_2: type fixed, parent world, child u_profile_2, origin xyz=0.6 0 0.05 rpy=0 0 0
- joint world_to_obstacle: origin xyz=0.71 0 0.015 rpy=0 0 0 -> xyz=0.85 0 0.005 rpy=0 0 0
- joint world_to_side_1: origin xyz=0.75 0.2 0.0275 rpy=0 0 0 -> xyz=0.85 0.2 0.0275 rpy=0 0 0
- joint world_to_side_2: origin xyz=0.75 -0.2 0.0275 rpy=0 0 0 -> xyz=0.85 -0.2 0.0275 rpy=0 0 0
- joint world_to_table: origin xyz=0.85 0 -0.05 rpy=0 0 0 -> xyz=0.85 0 -0.005 rpy=0 0 0
- joint world_to_u_profile: origin xyz=0.985 0 0.105 rpy=0 0 0 -> xyz=1.1 0 0.05 rpy=0 0 0
