Commit message: publish work from python node works!

File: setup_1_support/urdf/setup_1.xacro (robot description, xacro)
@@ -47,7 +47,13 @@
     <origin xyz="0 0 0.01" rpy="0 0 0" />
 </joint>
+<link name="work" />
+<joint name="world_to_work" type="fixed">
+  <parent link="world"/>
+  <child link="work"/>
+  <origin xyz="0.8 -0.5 0" rpy="0 0 0" />
+</joint>
 <!-- Load a work object -->
 <!-- <xacro:include filename="$(find setup_1_support)/urdf/work/boxes.urdf" /> -->
-<xacro:include filename="$(find setup_1_support)/urdf/work/$(arg work)" />
+<!-- <xacro:include filename="$(find setup_1_support)/urdf/work/$(arg work)" /> -->
 <!-- <xacro:include filename="$(find setup_1_support)/urdf/work/l_profile.urdf" /> -->
 </robot>

File: setup_1_support/urdf/work/boxes.urdf (robot description, URDF)
Before this commit: robot table_with_blocks, 3 links, 3 joints
Links:
- added link world

File: setup_1_support/urdf/work/kingpin.urdf (robot description, URDF)
Before this commit: robot kingpin, 5 links, 5 joints
Links:
- added link world

File: setup_1_support/urdf/work/l_profile.urdf (robot description, URDF)
Before this commit: robot l_profile, 3 links, 3 joints
Joints:
- removed joint world_to_work

Commit message: cleanup publish_work a bit

File: setup_1_support/urdf/setup_1.xacro (robot description, xacro)
@@ -47,10 +47,10 @@
     <origin xyz="0 0 0.01" rpy="0 0 0" />
 </joint>
-<link name="work" />
+<!-- <link name="work" />
 <joint name="world_to_work" type="fixed">
   <parent link="world"/>
   <child link="work"/>
   <origin xyz="0.8 -0.5 0" rpy="0 0 0" />
-</joint>
+</joint> -->
 <!-- Load a work object -->
 <!-- <xacro:include filename="$(find setup_1_support)/urdf/work/boxes.urdf" /> -->

File: setup_1_support/urdf/work/l_profile.urdf (robot description, URDF)
Before this commit: robot l_profile, 3 links, 2 joints
Links:
- removed link work
- added link world
Joints:
- removed joint work_to_l_base
- added joint world_to_l_base: type fixed, parent world, child l_base, origin xyz=0.9 0 0.01 rpy=0 0 0

File: setup_1_support/urdf/work/nothing.urdf (robot description, URDF)
Before this commit: robot nothing, 1 links, 1 joints
Links:
- removed link work
- added link world
Joints:
- removed joint world_to_work

Commit message: add new torch and smaller box

File: setup_1_support/urdf/setup_1.xacro (robot description, xacro)
@@ -16,14 +16,14 @@
 <link name="torch">
     <visual>
-    <origin xyz="0 0 0" rpy="0 0 0"/>
+    <origin xyz="0.380 0 0" rpy="0 -0.78539816339 0"/>
         <geometry>
-            <mesh filename="package://setup_1_support/meshes/visual/torch.stl"  scale=".01 .01 .01"/>
+            <mesh filename="package://setup_1_support/meshes/visual/mig_torch_small.stl"  scale="1 1 1"/>
         </geometry>
         <material name="gray"/>
     </visual>
     <collision>
-    <origin xyz="0 0 0" rpy="0 0 0"/>
+    <origin xyz="0.380 0 0" rpy="0 -0.78539816339 0"/>
         <geometry>
-            <mesh filename="package://setup_1_support/meshes/collision/torch.stl"  scale=".01 .01 .01"/>
+            <mesh filename="package://setup_1_support/meshes/collision/mig_torch_small.stl"  scale="1 1 1"/>
         </geometry>
     </collision>
@@ -39,5 +39,5 @@
     <parent link="torch"/>
     <child link="torch_tip"/>
-    <origin xyz="0.315 0 0.035" rpy="0 2.3560569232 0" />
+    <origin xyz="0.380 0 0" rpy="0 2.3560569232 0" />
 </joint>
 <!-- weld tip offset from workpiece -->
@@ -45,5 +45,5 @@
     <parent link="torch_tip"/>
     <child link="tool_tip"/>
-    <origin xyz="0 0 0.01" rpy="0 0 0" />
+    <origin xyz="0 0 0.02" rpy="0 0 0" />
 </joint>
 <!-- <link name="work" />

File: setup_3_support/urdf/work/halfopen_box.urdf (robot description, URDF)
Before this commit: robot halfopen_box, 2 links, 1 joints
Links:
- link wobj: geometry collision mesh filename=halfopen_box_small.stl scale=.001 .001 .001; visual mesh filename=halfopen_box_small.stl scale=.001 .001 .001
