Commit message: add l profile with obstacle as separat urdf

File: setup_1_support/urdf/work/l_profile_obstacle.urdf (robot description, URDF)
Before this commit: robot l_profile, 3 links, 2 joints
Links:
- added link obstacle; collision box size=0.1 0.1 0.04; visual box size=0.1 0.1 0.05
Joints:
- added joint l_base_to_obstacle: type fixed, parent l_base, child obstacle, origin xyz=-0.02 0 0.045 rpy=0 0 0
