Commit message: add obstacle to l_profile

File: setup_1_support/urdf/work/l_profile.urdf (robot description, URDF)
Before this commit: robot l_profile, 3 links, 2 joints
Links:
- added link obstacle; collision box size=0.1 0.02 0.04; visual box size=0.1 0.02 0.05
Joints:
- added joint l_base_to_obstacle: type fixed, parent l_base, child obstacle, origin xyz=-0.02 0 0.045 rpy=0 0 0

Commit message: remove submodule and random changes because aaargh

File: setup_1_support/urdf/work/l_profile.urdf (robot description, URDF)
Before this commit: robot l_profile, 4 links, 3 joints
Links:
- removed link obstacle
Joints:
- removed joint l_base_to_obstacle

File: setup_3_support/urdf/work/halfopen_box.urdf (robot description, URDF)
Before this commit: robot halfopen_box, 2 links, 1 joints
Links:
- link wobj: geometry collision box size=0.01 0.01 0.01; visual box size=0.01 0.01 0.01

Commit message: add floor plate to l_profile case

File: setup_1_support/urdf/work/l_profile.urdf (robot description, URDF)
Before this commit: robot l_profile, 3 links, 2 joints
Links:
- added link floor; collision box size=2 2 0.02; visual box size=2 2 0.02
Joints:
- added joint world_to_floor: type fixed, parent world, child floor, origin xyz=1 0 -0.02 rpy=0 0 0

File: setup_1_support/urdf/work/l_profile_obstacle.urdf (robot description, URDF)
Before this commit: robot l_profile_obstacle, 4 links, 3 joints
Links:
- added link floor; collision box size=2 2 0.02; visual box size=2 2 0.02
Joints:
- added joint world_to_floor: type fixed, parent world, child floor, origin xyz=1 0 -0.02 rpy=0 0 0
